Commit message: Added rail to ur10
Signed-off-by: Juancams <jc.manzanares.serrano@gmail.com>

File: urdf/ur.ros2_control.xacro (robot description, xacro)
@@ -157,4 +157,11 @@
           <param name="initial_value">${initial_positions['wrist_3_joint']}</param>
         </state_interface>
+        <state_interface name="velocity"/>
+        <state_interface name="effort"/>
+      </joint>
+      <joint name="${tf_prefix}rail_joint">
+        <command_interface name="position"/>
+        <command_interface name="velocity"/>
+        <state_interface name="position"/>
         <state_interface name="velocity"/>
         <state_interface name="effort"/>

File: urdf/ur.urdf.xacro (robot description, xacro)
@@ -95,5 +95,5 @@
     trajectory_port="$(arg trajectory_port)"
   >
-    <origin xyz="0 1.5 0" rpy="0 0 0" />          <!-- position robot in the world -->
+    <origin xyz="-1.8 -1.6 0.7" rpy="0 0 0" />          <!-- position robot in the world -->
   </xacro:ur_robot>
   <!-- arm ur10-->
@@ -134,6 +134,7 @@
     script_sender_port="$(arg script_sender_port)"
     trajectory_port="$(arg trajectory_port)"
+    generate_base="true"
   >
-    <origin xyz="0 -1.5 0" rpy="0 0 0" />          <!-- position robot in the world -->
+    <origin xyz="0 -2.39 1" rpy="-1.56 0 0" />          <!-- position robot in the world -->
   </xacro:ur_robot>
   <xacro:sensor_d435i name="ur5_camera" parent="ur5_wrist_3_link" use_nominal_extrinsics="true">

File: urdf/ur_macro.xacro (robot description, xacro)
@@ -83,5 +83,6 @@
     trajectory_port:=50003
     non_blocking_read:=true
-    keep_alive_count:=2"
+    keep_alive_count:=2
+    generate_base:=false"
     >
     <!-- Load configuration data from the provided .yaml files -->
@@ -255,10 +256,47 @@
       </xacro:cylinder_inertial>
     </link>
-    <!-- base_joint fixes base_link to the environment -->
-    <joint name="${tf_prefix}base_joint" type="fixed">
-      <xacro:insert_block name="origin" />
-      <parent link="${parent}" />
-      <child link="${tf_prefix}base_link" />
-    </joint>
+    <xacro:if value="${generate_base}">
+      <link name="${tf_prefix}rail_link">
+        <visual>
+          <origin xyz="0 0 0" rpy="0 0 0"/>
+          <geometry>
+            <box size="2 0.2 0.1"/>
+          </geometry>
+        </visual>
+        <collision>
+          <origin xyz="0 0 0" rpy="0 0 0"/>
+          <geometry>
+            <box size="2 0.2 0.1"/>
+          </geometry>
+        </collision>
+        <inertial>
+          <origin xyz="0 0 -0.1" rpy="0 0 0"/>
+          <mass value="10.0"/>
+          <inertia ixx="0.1" ixy="0.0" ixz="0.0" iyy="0.1" iyz="0.0" izz="0.1"/>
+        </inertial>
+      </link>
+    </xacro:if>
+    <!-- base_joint fixes base to the environment -->
+    <xacro:unless value="${generate_base}">
+      <joint name="${tf_prefix}base_joint" type="fixed">
+        <xacro:insert_block name="origin" />
+        <parent link="${parent}" />
+        <child link="${tf_prefix}base_link" />
+      </joint>
+    </xacro:unless>
+    <xacro:if value="${generate_base}">
+      <joint name="${tf_prefix}base_joint" type="fixed">
+        <xacro:insert_block name="origin" />
+        <parent link="${parent}" />
+        <child link="${tf_prefix}rail_link" />
+      </joint>
+      <joint name="${tf_prefix}rail_joint" type="prismatic">
+        <parent link="${tf_prefix}rail_link"/>
+        <child link="${tf_prefix}base_link"/>
+        <origin xyz="0 0 0.05" rpy="0 0 0"/>
+        <axis xyz="1 0 0"/>
+        <limit lower="-1.0" upper="1.0" effort="10" velocity="0.1"/>
+      </joint>
+    </xacro:if>
     <!-- joints - main serial chain -->
     <joint name="${tf_prefix}base_link-base_link_inertia" type="fixed">
